File: InputStage.kicad_sch (KiCad schematic)
At the start: 5 parts, among them J2 NMJ4HCD2, U1 TL072

Commit message: using smt caps and resistors
Parts:
- C1: footprint ECE319K:C_Axial_200mil -> Capacitor_SMD:C_0805_2012Metric_Pad1.18x1.45mm_HandSolder
- R1, R2: footprint Resistor_THT:R_Axial_DIN0207_L6.3mm_D2.5mm_P10.16mm_Horizontal -> Resistor_SMD:R_0805_2012Metric_Pad1.20x1.40mm_HandSolder
Changed lines of the file:
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@@
 			)
 		)
-		(property "Footprint" "Resistor_THT:R_Axial_DIN0207_L6.3mm_D2.5mm_P10.16mm_Horizontal"
+		(property "Footprint" "Resistor_SMD:R_0805_2012Metric_Pad1.20x1.40mm_HandSolder"
 			(at 67.31 93.853 90)
 			(effects
@@
 			)
 		)
-		(property "Footprint" "ECE319K:C_Axial_200mil"
+		(property "Footprint" "Capacitor_SMD:C_0805_2012Metric_Pad1.18x1.45mm_HandSolder"
 			(at 82.55 91.1098 0)
 			(effects
@@
 			)
 		)
-		(property "Footprint" "Resistor_THT:R_Axial_DIN0207_L6.3mm_D2.5mm_P10.16mm_Horizontal"
+		(property "Footprint" "Resistor_SMD:R_0805_2012Metric_Pad1.20x1.40mm_HandSolder"
 			(at 90.043 101.6 90)
 			(effects

Commit message: change metal film resistor footprint
Parts:
- U1: footprint ECE319K:DIP-8_W7.62mm_LongPads -> Package_SO:SO-8_3.9x4.9mm_P1.27mm
Changed lines of the file:
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@@
 			)
 		)
-		(property "Footprint" "ECE319K:DIP-8_W7.62mm_LongPads"
+		(property "Footprint" "Package_SO:SO-8_3.9x4.9mm_P1.27mm"
 			(at 98.425 89.535 0)
 			(effects
@@
 			)
 		)
-		(property "Footprint" "ECE319K:DIP-8_W7.62mm_LongPads"
+		(property "Footprint" "Package_SO:SO-8_3.9x4.9mm_P1.27mm"
 			(at 100.965 107.95 0)
 			(effects

Commit message: initial layout
Parts:
- J2: value NMJ4HCD2 -> NMJ4HCD2_input
Changed lines of the file:
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@@
 			)
 		)
-		(property "Value" "NMJ4HCD2"
+		(property "Value" "NMJ4HCD2_input"
 			(at 53.34 83.82 0)
 			(effects
