File: OutputStage.kicad_sch (KiCad schematic)
At the start: 8 parts, among them J4 NMJ4HCD2, SW1 SW_DPDT_x2

Commit message: using smt caps and resistors
Parts:
- C22: footprint ECE319K:C_Axial_200mil -> Capacitor_SMD:C_0805_2012Metric_Pad1.18x1.45mm_HandSolder
- R26, R27, R28, R29: footprint Resistor_THT:R_Axial_DIN0207_L6.3mm_D2.5mm_P10.16mm_Horizontal -> Resistor_SMD:R_0805_2012Metric_Pad1.20x1.40mm_HandSolder
Changed lines of the file:
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@@
 			)
 		)
-		(property "Footprint" "Resistor_THT:R_Axial_DIN0207_L6.3mm_D2.5mm_P10.16mm_Horizontal"
+		(property "Footprint" "Resistor_SMD:R_0805_2012Metric_Pad1.20x1.40mm_HandSolder"
 			(at 99.695 115.697 90)
 			(effects
@@
 			)
 		)
-		(property "Footprint" "Resistor_THT:R_Axial_DIN0207_L6.3mm_D2.5mm_P10.16mm_Horizontal"
+		(property "Footprint" "Resistor_SMD:R_0805_2012Metric_Pad1.20x1.40mm_HandSolder"
 			(at 151.003 137.16 90)
 			(effects
@@
 			)
 		)
-		(property "Footprint" "Resistor_THT:R_Axial_DIN0207_L6.3mm_D2.5mm_P10.16mm_Horizontal"
+		(property "Footprint" "Resistor_SMD:R_0805_2012Metric_Pad1.20x1.40mm_HandSolder"
 			(at 127.635 136.652 90)
 			(effects
@@
 			)
 		)
-		(property "Footprint" "ECE319K:C_Axial_200mil"
+		(property "Footprint" "Capacitor_SMD:C_0805_2012Metric_Pad1.18x1.45mm_HandSolder"
 			(at 91.44 116.5098 0)
 			(effects
@@
 			)
 		)
-		(property "Footprint" "Resistor_THT:R_Axial_DIN0207_L6.3mm_D2.5mm_P10.16mm_Horizontal"
+		(property "Footprint" "Resistor_SMD:R_0805_2012Metric_Pad1.20x1.40mm_HandSolder"
 			(at 127.635 106.172 90)
 			(effects

Commit message: change metal film resistor footprint
Parts:
- renumbered RV2 to Level_RV2
Changed lines of the file:
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@@
 		(dnp no)
 		(fields_autoplaced yes)
-		(property "Reference" "RV2"
+		(property "Reference" "Level_RV2"
 			(at 106.68 125.0949 0)
 			(effects
@@
 			(project "KlonePedal"
 				(path "/9e3f79d9-06b6-4799-a8c0-00f1612ca30b/e6f1a508-7b78-483d-9586-fd067ae996be"
-					(reference "RV2")
+					(reference "Level_RV2")
 					(unit 1)
 				)

Commit message: initial layout
Parts:
- removed SW1: SW_DPDT_x2, Connector_Wire:SolderWire-0.1sqmm_1x03_P3.6mm_D0.4mm_OD1mm, symbol Switch:SW_DPDT_x2
- added J5: SW1A_DPDT_x2, Connector_JST:JST_XH_S3B-XH-A_1x03_P2.50mm_Horizontal, symbol Connector_Generic:Conn_01x03
- J4: value NMJ4HCD2 -> NMJ4HCD2_output
Connections:
- net BypassSignal: now also J5.3 (Pin_3)
- net at Level_RV2.2, R27.2: now also J5.1 (Pin_1)
- net at J4.T, R27.1, R28.1: now also J5.2 (Pin_2)
Other:
- note added: "1"
- note added: "2"
- note added: "3"
Changed lines of the file:
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@@
 	(generator_version "9.0")
 	(paper "A4")
+	(text "1"
+		(exclude_from_sim no)
+		(at 119.888 127.762 0)
+		(effects
+			(font
+				(size 1.27 1.27)
+			)
+		)
+	)
+	(text "3"
+		(exclude_from_sim no)
+		(at 119.888 120.396 0)
+		(effects
+			(font
+				(size 1.27 1.27)
+			)
+		)
+	)
 	(text "Level"
 		(exclude_from_sim no)
@@
 		)
 	)
+	(text "2"
+		(exclude_from_sim no)
+		(at 133.604 125.222 0)
+		(effects
+			(font
+				(size 1.27 1.27)
+			)
+		)
+	)
 	(junction
 		(at 116.84 107.95)
@@
 	(wire
 		(pts
-			(xy 139.065 123.825) (xy 132.715 123.825)
-		)
-		(stroke
-			(width 0)
-			(type default)
-		)
-	)
-	(wire
-		(pts
 			(xy 108.585 117.475) (xy 108.585 122.555)
 		)
@@
 	(wire
 		(pts
+			(xy 122.555 128.27) (xy 130.81 128.27)
+		)
+		(stroke
+			(width 0)
+			(type default)
+		)
+	)
+	(wire
+		(pts
 			(xy 79.375 117.475) (xy 83.82 117.475)
 		)
@@
 	(wire
 		(pts
+			(xy 122.555 126.365) (xy 122.555 128.27)
+		)
+		(stroke
+			(width 0)
+			(type default)
+		)
+	)
+	(wire
+		(pts
 			(xy 112.395 126.365) (xy 116.84 126.365)
 		)
@@
 	(wire
 		(pts
+			(xy 122.555 119.38) (xy 130.81 119.38)
+		)
+		(stroke
+			(width 0)
+			(type default)
+		)
+	)
+	(wire
+		(pts
 			(xy 91.44 117.475) (xy 95.885 117.475)
 		)
@@
 	(wire
 		(pts
+			(xy 122.555 121.285) (xy 122.555 119.38)
+		)
+		(stroke
+			(width 0)
+			(type default)
+		)
+	)
+	(wire
+		(pts
 			(xy 108.585 130.175) (xy 108.585 134.62)
 		)
@@
 	(wire
 		(pts
+			(xy 130.81 119.38) (xy 130.81 121.285)
+		)
+		(stroke
+			(width 0)
+			(type default)
+		)
+	)
+	(wire
+		(pts
 			(xy 116.84 126.365) (xy 122.555 126.365)
+		)
+		(stroke
+			(width 0)
+			(type default)
+		)
+	)
+	(wire
+		(pts
+			(xy 130.81 123.825) (xy 139.065 123.825)
+		)
+		(stroke
+			(width 0)
+			(type default)
+		)
+	)
+	(wire
+		(pts
+			(xy 130.81 128.27) (xy 130.81 126.365)
 		)
 		(stroke
@@
 	)
 	(symbol
-		(lib_id "Switch:SW_DPDT_x2")
-		(at 127.635 123.825 180)
+		(lib_id "Connector_Audio:NMJ4HCD2")
+		(at 161.29 123.825 180)
 		(unit 1)
 		(exclude_from_sim no)
@@
 		(dnp no)
 		(fields_autoplaced yes)
-		(property "Reference" "SW1"
-			(at 127.635 114.935 0)
-			(effects
-				(font
-					(size 1.27 1.27)
-				)
-			)
-		)
-		(property "Value" "SW_DPDT_x2"
-			(at 127.635 117.475 0)
-			(effects
-				(font
-					(size 1.27 1.27)
-				)
-			)
-		)
-		(property "Footprint" "Connector_Wire:SolderWire-0.1sqmm_1x03_P3.6mm_D0.4mm_OD1mm"
-			(at 127.635 123.825 0)
-			(effects
-				(font
-					(size 1.27 1.27)
-				)
-				(hide yes)
-			)
-		)
-		(property "Datasheet" "~"
-			(at 127.635 123.825 0)
-			(effects
-				(font
-					(size 1.27 1.27)
-				)
-				(hide yes)
-			)
-		)
-		(property "Description" "Switch, dual pole double throw, separate symbols"
-			(at 127.635 123.825 0)
-			(effects
-				(font
-					(size 1.27 1.27)
-				)
-				(hide yes)
-			)
-		)
-		(pin "2"
-		)
-		(pin "1"
-		)
-		(pin "3"
-		)
-		(pin "5"
-		)
-		(pin "4"
-		)
-		(pin "6"
-		)
-		(instances
-			(project ""
-				(path "/9e3f79d9-06b6-4799-a8c0-00f1612ca30b/e6f1a508-7b78-483d-9586-fd067ae996be"
-					(reference "SW1")
-					(unit 1)
-				)
-			)
-		)
-	)
-	(symbol
-		(lib_id "Connector_Audio:NMJ4HCD2")
-		(at 161.29 123.825 180)
-		(unit 1)
-		(exclude_from_sim no)
-		(in_bom yes)
-		(on_board yes)
-		(dnp no)
-		(fields_autoplaced yes)
 		(property "Reference" "J4"
-			(at 167.005 123.8249 0)
+			(at 166.37 123.8249 0)
 			(effects
 				(font
@@
 			)
 		)
-		(property "Value" "NMJ4HCD2"
-			(at 167.005 126.3649 0)
+		(property "Value" "NMJ4HCD2_output"
+			(at 166.37 126.3649 0)
 			(effects
 				(font
@@
 					(unit 1)
 				)
+			)
+		)
+	)
+	(symbol
+		(lib_id "Connector_Generic:Conn_01x03")
+		(at 125.73 123.825 180)
+		(unit 1)
+		(exclude_from_sim no)
+		(in_bom yes)
+		(on_board yes)
+		(dnp no)
+		(fields_autoplaced yes)
+		(property "Reference" "J5"
+			(at 125.73 114.935 0)
+			(effects
+				(font
+					(size 1.27 1.27)
+				)
+			)
+		)
+		(property "Value" "SW1A_DPDT_x2"
+			(at 125.73 117.475 0)
+			(effects
+				(font
+					(size 1.27 1.27)
+				)
+			)
+		)
+		(property "Footprint" "Connector_JST:JST_XH_S3B-XH-A_1x03_P2.50mm_Horizontal"
+			(at 125.73 123.825 0)
+			(effects
+				(font
+					(size 1.27 1.27)
+				)
+				(hide yes)
+			)
+		)
+		(property "Datasheet" "~"
+			(at 125.73 123.825 0)
+			(effects
+				(font
+					(size 1.27 1.27)
+				)
+				(hide yes)
+			)
+		)
+		(property "Description" "Generic connector, single row, 01x03, script generated (kicad-library-utils/schlib/autogen/connector/)"
+			(at 125.73 123.825 0)
+			(effects
+				(font
+					(size 1.27 1.27)
+				)
+				(hide yes)
+			)
+		)
+		(pin "1"
+		)
+		(pin "2"
+		)
+		(pin "3"
+		)
+		(instances
+			(project "KlonePedal"
+				(path "/9e3f79d9-06b6-4799-a8c0-00f1612ca30b/e6f1a508-7b78-483d-9586-fd067ae996be"
+					(reference "J5")
+					(unit 1)
+				)
